File: Hardware/Bike/Bike.kicad_sch (KiCad schematic)
At the start: 18 parts, among them U1 ESP32-WROOM-32

Commit message: schematics design
Parts:
- removed D1: LED1, symbol Device:LED
- removed D2: LED2, symbol Device:LED
- removed D4: LED4, symbol Device:LED
- removed D5: LED5, symbol Device:LED
- removed D6: LED6, symbol Device:LED
- removed Power_Sw: ~, symbol Switch:SW_SPST
- removed R1, R2, R3, R4, R5, R6: 1k, symbol Device:R
- removed U1: ESP32-WROOM-32, RF_Module:ESP32-WROOM-32, symbol RF_Module:ESP32-WROOM-32
- removed U2: ~, symbol Bike Project:NEO-6M-GPS
- removed U3: ~, symbol RGB-LED:_WS2812B-MINI
- removed U4: ~, symbol 2Digit-7Seg:SMC562LB
- removed U5: ~, symbol MLT-5020:MLT-5020
- added BZ1: Buzzer, Buzzer_Beeper:Buzzer_CUI_CPT-9019S-SMT, symbol Device:Buzzer
- added C1, C2, C4, C5, C9: 10uF, Capacitor_SMD:C_0402_1005Metric, symbol Device:C_Small
- added C3, C8: 1uF, Capacitor_SMD:C_0402_1005Metric, symbol Device:C_Small
- added D1: MBR120, symbol Device:D_Schottky_Dual_CommonAnode_KAK_Split
- added D10, D11, D12, D8, D9: LED1, symbol Device:LED
- added D2: RED, LED_SMD:LED_0402_1005Metric, symbol Device:LED_Small
- added D4: CHG, LED_SMD:LED_0402_1005Metric, symbol Device:LED_Small
- added D5, D6, D7: LESD5D5, Diode_SMD:D_SOD-523, symbol Diode:ESD5Zxx
- added J1: SW1, symbol Connector:Conn_01x02_Socket
- added J3: GPS, Connector_PinSocket_2.54mm:PinSocket_1x04_P2.54mm_Vertical, symbol Connector:Conn_01x04_Socket
- added J4: BAT, symbol Connector:Conn_01x02_Socket
- added J5: ON, symbol Connector:Conn_01x02_Socket
- added J7: USB_C_Receptacle, Connector_USB:USB_C_Receptacle_Molex_105450-0101, symbol Connector:USB_C_Receptacle
- added LED1: 19-037A/RSGHBHW1-S03/2T, EXT_LIB:LED-ARRAY-SMD_4P-L1.6-W1.6-TR_EVERLIGHT_RSGHBHW1-S03, symbol RGBA_0606:19-037A_RSGHBHW1-S03_2T
- added Q1: DMG3415U, symbol Device:Q_PMOS_GDS
- added Q2, Q3, Q4: NPN, symbol Simulation_SPICE:NPN
- added R1, R15, R16, R17, R3: 100K, Resistor_SMD:R_0402_1005Metric_Pad0.72x0.64mm_HandSolder, symbol Device:R_Small
- added R10, R22, R23, R24, R4, R6, R9: 1k, Resistor_SMD:R_0402_1005Metric_Pad0.72x0.64mm_HandSolder, symbol Device:R_Small
- added R11, R5: 1K, Resistor_SMD:R_0402_1005Metric_Pad0.72x0.64mm_HandSolder, symbol Device:R_Small
- added R12: 150, Resistor_SMD:R_0402_1005Metric, symbol Device:R_Small
- added R13, R14, R8: 100, Resistor_SMD:R_0402_1005Metric, symbol Device:R_Small
- added R18, R19: 5.1K-1%, Resistor_SMD:R_0402_1005Metric_Pad0.72x0.64mm_HandSolder, symbol Device:R_Small
- added R2, R20, R21: 10K, Resistor_SMD:R_0402_1005Metric_Pad0.72x0.64mm_HandSolder, symbol Device:R_Small
- added R7: 4.7K, Resistor_SMD:R_0402_1005Metric_Pad0.72x0.64mm_HandSolder, symbol Device:R_Small
- added SW1: RST, symbol Switch:SW_Push
- added U1: ESP32-WROOM-32-N4, ESP32-WROOM-32:MOD_ESP32-WROOM-32_EXP, symbol ESP32-WROOM-32-N4:ESP32-WROOM-32-N4
- added U2: AP2112K-3.3, Package_TO_SOT_SMD:SOT-23-5, symbol Regulator_Linear:AP2112K-3.3
- added U3: MCP73831-2-OT, Package_TO_SOT_SMD:SOT-23-5, symbol Battery_Management:MCP73831-2-OT
- added U5: CP2104, Package_DFN_QFN:QFN-24-1EP_4x4mm_P0.5mm_EP2.6x2.6mm, symbol Interface_USB:CP2104
- D3: value LED3 -> LED1
Connections:
- net GND: now also C1.2, C2.2, C3.2, C4.2, C5.2, C8.2, C9.2, D2.1 (K), D5.1 (K), D6.1 (K), D7.1 (K), J1.2 (Pin_2), J3.4 (Pin_4), J4.1 (Pin_1), J7.A1 (GND), J7.A12 (GND), J7.B1 (GND), J7.B12 (GND), J7.S1 (SHIELD), Q2.3 (E), R1.2, R16.2, R18.2, R19.2, R7.2, SW1.1, U1.1 (GND), U1.15 (GND), U1.38 (GND), U1.39 (GND), U1.40 (GND), U1.41 (GND), U1.42 (GND), U1.43 (GND), U1.44 (GND), U1.45 (GND), U1.46 (GND), U1.47 (GND), U2.2 (GND), U3.2 (V_{SS}), U5.2 (GND), U5.25 (GND); no longer D3.1 (K)
- net LED1: now also R4.2, U1.11 (IO26)
- net LED2: now also R9.2, U1.12 (IO27)
- net LED3: now also R10.2, U1.13 (IO14)
- net LED4: now also R22.2, U1.14 (IO12)
- net LED5: now also R23.2, U1.16 (IO13)
- net LED6: now also R24.2, U1.23 (IO15)
- net +BATT: now reaches D3.2 (A)
- net +BATT: now also C5.1, D10.2 (A), D11.2 (A), D12.2 (A), D8.2 (A), D9.2 (A), J3.1 (Pin_1), J5.1 (Pin_1), LED1.4 (+), Q1.2 (D), R15.1, R8.1, U3.3 (V_{BAT})
- new net: BZ1.1 (+), R8.2
- new net: J4.2 (Pin_2), J5.2 (Pin_2)
- new net: Q4.2 (B), R21.2
- new net: D2.2 (A), R5.2
- new net: D3.1 (K), R4.1
- new net: D11.1 (K), R23.1
- new net: R7.1, U3.5 (PROG)
- new net: R11.1, U3.1 (STAT)
- new net: D9.1 (K), R10.1
- new net: J7.A5 (CC1), R18.1
- new net: C1.1, D1.1 (K), Q1.3 (S), R3.2, U2.1 (VIN)
- new net: R3.1, U2.3 (EN)
- new net: Q3.2 (B), R20.2
- new net: LED1.1 (R-), R12.2
- new net: D4.1 (K), R11.2
- new net: LED1.2 (G-), R13.2
- new net: LED1.3 (B-), R14.2
- new net: Q2.2 (B), R6.2
- new net: D8.1 (K), R9.1
- new net: D12.1 (K), R24.1
- new net: D10.1 (K), R22.1
- new net: BZ1.2 (-), Q2.1 (C)
- new net: J7.B5 (CC2), R19.1
- new net +3V3: C2.1, C3.1, C4.1, C9.1, R17.1, R2.1, U1.2 (3V3), U2.5 (VOUT), U5.5 (VIO), U5.6 (VDD), U5.7 (REGIN)
- new net BUZ: R6.1, U1.9 (IO33)
- new net DTR: Q3.3 (E), R21.1, U5.23 (~{DTR})
- new net ESP-RST: C8.1, Q4.1 (C), R17.2, SW1.2, U1.3 (EN)
- new net GPIO0: Q3.1 (C), U1.25 (IO0)
- new net GPIO2: U1.24 (IO2)
- new net GPS_RX: J3.3 (Pin_3)
- new net GPS_TX: J3.2 (Pin_2)
- new net LED_B: R14.1
- new net LED_G: R13.1
- new net LED_R: R12.1
- new net RAD_RX: U1.27 (IO16)
- new net RAD_TX: U1.28 (IO17)
- new net RTS: Q4.3 (E), R20.1, U5.19 (~{RTS})
- new net RX0: U1.34 (RXD0), U5.21 (TXD)
- new net STATUS: R5.1, U1.6 (IO34)
- new net SW1_IN: J1.1 (Pin_1), R2.2, U1.10 (IO25)
- new net TX0: U1.35 (TXD0), U5.20 (RXD)
- new net USB_N: D6.2 (A), J7.A7 (D-), J7.B7 (D-), U5.4 (D-)
- new net USB_P: D7.2 (A), J7.A6 (D+), J7.B6 (D+), U5.3 (D+)
- new net VBAT_SEN: R15.2, R16.1, U1.7 (IO35)
- new net VBUS: D1.2 (A), D4.2 (A), D5.2 (A), J7.A4 (VBUS), J7.A9 (VBUS), J7.B4 (VBUS), J7.B9 (VBUS), Q1.1 (G), R1.1, U3.4 (V_{DD}), U5.8 (VBUS)
- no-connect marks 0 -> 10
Other:
- note added: "BAT CHARGER"
- note added: "Current Limit"
- note added: "ESP32-D0WDQ6"
- note added: "GPS EXTERNAL MODULE"
- note added: "PCB SIZE: 50 x 55 mm"
- note added: "POWER IN + FILTERING"
- note added: "Serial2"
- note added: "USB_C TO TTL"
- note added: "WHERE IS PLACED ?"
- note removed: "1-Actively pull EN pin low briefly to trigger reset."
- note removed: "2-After reset, during strapping pin reading process : active pull IO0 pin low & make sure IO2 remains low."
- note removed: "3-Esp32 begins in download boot mode"
- note removed: "4-Begin communicating your code via UART to ESP memory"
- note removed: "5-Trigger another reset and ensure IO0 is high"
- note removed: "6- Battery needs to be( 3.7V , 1500mAh )"
- note removed: "7- Battry charges from the USB_Type_c Port."
- note removed: "Notes Before Flashing Code:"
