File: Hardware/Bike/Bike.kicad_sch (KiCad schematic)
At the start: 67 parts, among them J1 BAT, J3 SW1, J4 BUZ, J5 GPS, J7 ON, Q1 DMG3415U, Q2 Q_NPN_BEC, Q8 LMUN5214DW1T1G, SW1 RST, U1 APTD3216SECK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

Commit message: pcb fix again
Other:
- moved on the sheet: C11
Changed lines of the file:
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@@
 	)
 	(junction
+		(at 157.48 35.56)
+		(diameter 0)
+		(color 0 0 0 0)
+	)
+	(junction
 		(at 241.3 64.77)
 		(diameter 0)
@@
 		(color 0 0 0 0)
 	)
-	(junction
-		(at 158.75 35.56)
-		(diameter 0)
-		(color 0 0 0 0)
-	)
 	(no_connect
 		(at 254 101.6)
@@
 	(wire
 		(pts
-			(xy 158.75 35.56) (xy 158.75 40.64)
-		)
-		(stroke
-			(width 0)
-			(type default)
-		)
-	)
-	(wire
-		(pts
-			(xy 158.75 35.56) (xy 161.29 35.56)
+			(xy 157.48 35.56) (xy 157.48 40.64)
 		)
 		(stroke
@@
 	(wire
 		(pts
-			(xy 152.4 35.56) (xy 158.75 35.56)
+			(xy 153.67 35.56) (xy 157.48 35.56)
 		)
 		(stroke
@@
 	(wire
 		(pts
-			(xy 152.4 38.1) (xy 152.4 35.56)
+			(xy 153.67 38.1) (xy 153.67 35.56)
 		)
 		(stroke
@@
 	(wire
 		(pts
+			(xy 157.48 35.56) (xy 161.29 35.56)
+		)
+		(stroke
+			(width 0)
+			(type default)
+		)
+	)
+	(wire
+		(pts
 			(xy 256.54 31.75) (xy 257.81 31.75)
 		)
@@
 	(wire
 		(pts
-			(xy 158.75 45.72) (xy 161.29 45.72)
+			(xy 157.48 45.72) (xy 161.29 45.72)
 		)
 		(stroke
@@
 	(global_label "VBAT_SEN"
 		(shape input)
-		(at 152.4 38.1 270)
+		(at 153.67 38.1 270)
 		(fields_autoplaced yes)
 		(effects
@@
 		)
 		(property "Intersheetrefs" "${INTERSHEET_REFS}"
-			(at 152.4 50.6326 90)
+			(at 153.67 50.6326 90)
 			(effects
 				(font
@@
 	(symbol
 		(lib_id "Device:C_Small")
-		(at 158.75 43.18 180)
+		(at 157.48 43.18 180)
 		(unit 1)
 		(exclude_from_sim no)
@@
 		(dnp no)
 		(property "Reference" "C11"
-			(at 157.48 44.704 90)
+			(at 157.734 46.228 90)
 			(effects
 				(font
@@
 		)
 		(property "Value" "100n"
-			(at 158.75 41.148 0)
+			(at 158.496 37.338 90)
 			(effects
 				(font
@@
 		)
 		(property "Footprint" "Capacitor_SMD:C_0402_1005Metric"
-			(at 158.75 43.18 0)
+			(at 157.48 43.18 0)
 			(effects
 				(font
@@
 		)
 		(property "Datasheet" "~"
-			(at 158.75 43.18 0)
+			(at 157.48 43.18 0)
 			(effects
 				(font
@@
 		)
 		(property "Description" "Unpolarized capacitor, small symbol"
-			(at 158.75 43.18 0)
+			(at 157.48 43.18 0)
 			(effects
 				(font
@@
 		)
 		(property "LCSC" ""
-			(at 158.75 43.18 0)
+			(at 157.48 43.18 0)
 			(effects
 				(font
