File: Hardware/Bike/Bike.kicad_pcb (KiCad board)
At the start: 4 copper layers, 54 x 35 mm, 70 parts, among them J1 BAT, J3 SW1, J4 BUZ, J5 GPS, J7 ON, Q1 DMG3415U, Q4 NPN, Q5 DMG3415U, Q6 DMG3415U, Q8 LMUN5214DW1T1G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

Commit message: fixing testing note
Parts:
- removed Q4: NPN, Package_TO_SOT_SMD:SOT-23
- removed Q5, Q6: DMG3415U, Package_TO_SOT_SMD:SOT-23
- removed R26, R27: 1k, Resistor_SMD:R_0402_1005Metric_Pad0.72x0.64mm_HandSolder
- removed RST: RST, Connector_PinSocket_2.54mm:PinSocket_1x02_P2.54mm_Vertical
- added C11: 100n, Capacitor_SMD:C_0402_1005Metric, B.Cu at (122.0, 131.1)
- added Q2: Q_NPN_BEC, Package_TO_SOT_SMD:SOT-23-3, B.Cu at (141.5, 129.0)
- added SW1: RST, Connector_PinSocket_2.54mm:PinSocket_1x02_P2.54mm_Vertical, F.Cu at (143.7, 103.1)
- moved R32 0.17 mm to (142.7, 127.7)
Connections:
- LED2 pad 10: Net-(LED2-DIG1) -> /DIG1_EN
- LED2 pad 5: Net-(LED2-DIG2) -> /DIG2_EN
Routing:
- net GND: track 119.9 -> 139.5 mm
- net +3V3: track 135.9 -> 119.2 mm
- net Net-(LED2-DIG1): track 14.2 -> 0.00 mm, vias 1 -> 0
- net Net-(LED2-DIG2): track 13.2 -> 0.00 mm, vias 1 -> 0
- net VBAT_SEN: track 51.0 -> 52.6 mm
- net Net-(J4-Pin_2): track 8.25 -> 7.12 mm
- net /DIG1_EN: track 42.2 -> 43.3 mm
- net Net-(Q2-B): track 2.70 -> 1.65 mm
- net /DIG2_EN: track 22.2 -> 22.1 mm, vias 1 -> 2

Commit message: pcb fix again
Routing:
- net +BATT: track 93.0 -> 90.7 mm
- net Net-(D1A-K): track 32.2 -> 30.6 mm
Changed lines of the file:
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@@
 		)
 		(property "Value" "DMG3415U"
-			(at 0 -2.4 90)
+			(at 0 -2.4 -90)
 			(layer "B.Fab")
 			(effects
@@
 			)
 		)
-		(sheetname "Root")
-		(sheetfile "Bike.kicad_sch")
 		(attr smd)
 		(fp_line
@@
 		)
 		(fp_text user "${REFERENCE}"
-			(at 0 0 90)
+			(at 0 0 -90)
 			(layer "B.Fab")
 			(effects
@@
 		)
 		(pad "2" smd roundrect
-			(at -0.9375 -0.95 270)
+			(at 0.9375 0 270)
 			(size 1.475 0.6)
 			(layers "B.Cu" "B.Paste" "B.Mask")
@@
 		)
 		(pad "3" smd roundrect
-			(at 0.9375 0 270)
+			(at -0.9375 -0.95 270)
 			(size 1.475 0.6)
 			(layers "B.Cu" "B.Paste" "B.Mask")
@@
 	)
 	(segment
+		(start 123.942893 127.927107)
+		(end 123.942893 130.367107)
+		(width 0.3)
+		(layer "B.Cu")
+		(net 57)
+	)
+	(segment
 		(start 115.772893 126.007107)
 		(end 115.272893 126.507107)
@@
 	)
 	(segment
-		(start 124.917893 128.762868)
-		(end 123.512893 130.167868)
+		(start 123.942893 130.367107)
+		(end 123.512893 130.797107)
 		(width 0.3)
 		(layer "B.Cu")
@@
 	)
 	(segment
-		(start 124.917893 126.027107)
-		(end 124.917893 128.762868)
+		(start 142.792893 125.272107)
+		(end 146.587893 125.272107)
 		(width 0.3)
 		(layer "B.Cu")
@@
 	)
 	(segment
-		(start 142.792893 125.272107)
-		(end 146.587893 125.272107)
+		(start 123.967893 127.902107)
+		(end 123.942893 127.927107)
 		(width 0.3)
 		(layer "B.Cu")
@@
 	)
 	(segment
-		(start 123.512893 130.167868)
-		(end 123.512893 130.797107)
-		(width 0.3)
-		(layer "B.Cu")
-		(net 57)
-	)
-	(segment
 		(start 116.842893 126.007107)
 		(end 115.772893 126.007107)
@@
 	)
 	(segment
+		(start 124.917893 124.907107)
+		(end 124.917893 126.027107)
+		(width 0.3)
+		(layer "B.Cu")
+		(net 58)
+	)
+	(segment
+		(start 125.292893 124.532107)
+		(end 124.917893 124.907107)
+		(width 0.3)
+		(layer "B.Cu")
+		(net 58)
+	)
+	(segment
 		(start 124.892893 124.257107)
 		(end 125.160393 124.257107)
@@
 	)
 	(segment
+		(start 125.292893 124.124607)
+		(end 125.292893 124.532107)
+		(width 0.3)
+		(layer "B.Cu")
+		(net 58)
+	)
+	(segment
 		(start 127.042893 123.119607)
 		(end 127.042893 121.857107)
@@
 		(width 0.3)
 		(layer "B.Cu")
-		(net 58)
-	)
-	(segment
-		(start 123.967893 127.902107)
-		(end 123.967893 124.332107)
-		(width 0.3)
-		(layer "B.Cu")
